File: PCB/ktRMT_Thumb.kicad_pcb (KiCad board)
At the start: 2 copper layers, 19.1 x 57.1 mm, 11 parts, among them SW1 SW_Push, SW2 SW_Push, U1 AD009-06H

Commit message: 2nd
Parts:
- removed C1, C2: 47uF/16V, Capacitor_SMD:C_1210_3225Metric
- U1: value AD009-06H -> HB1531E
Connections:
- SW1 pad 2: Net-(SW1-Pad2) -> Net-(U1-Pad11)
- SW2 pad 1: Net-(SW2-Pad1) -> Net-(U1-Pad10)
- U1 pad 10: unconnected-(U1-Pad10) -> Net-(U1-Pad10)
- U1 pad 11: unconnected-(U1-Pad11) -> Net-(U1-Pad11)
- U1 pad 12: unconnected-(U1-Pad12) -> Net-(SW1-Pad1)
- U1 pad 2: Net-(C2-Pad2) -> unconnected-(U1-Pad2)
- U1 pad 3: Net-(SW2-Pad2) -> unconnected-(U1-Pad3)
- U1 pad 4: Net-(SW2-Pad1) -> unconnected-(U1-Pad4)
- U1 pad 5: Net-(SW1-Pad2) -> unconnected-(U1-Pad5)
- U1 pad 6: Net-(SW1-Pad1) -> unconnected-(U1-Pad6)
- U1 pad 9: unconnected-(U1-Pad9) -> Net-(SW2-Pad2)
Routing:
- net Net-(SW2-Pad1): track 47.7 -> 0.00 mm, vias 3 -> 0
- net Net-(U1-Pad10): track 0.00 -> 44.8 mm, vias 0 -> 3
- net Net-(U1-Pad11): track 0.00 -> 30.9 mm, vias 0 -> 1
- net Net-(SW1-Pad2): track 30.3 -> 0.00 mm, vias 1 -> 0
- net Net-(BT1-Pad1): track 34.8 -> 17.2 mm
- net Net-(BT1-Pad2): track 35.7 -> 23.8 mm, vias 6 -> 5
- net Net-(SW1-Pad1): track 22.8 -> 30.4 mm
- net Net-(SW2-Pad2): track 49.1 -> 42.3 mm
- net Net-(C2-Pad2): track 5.36 -> 0.00 mm
