File: PCB/ktRMT_Thumb.kicad_sch (KiCad schematic)
At the start: 9 parts, among them SW1 SW_Push, SW2 SW_Push, U1 AD009-06H

Commit message: 2nd
Parts:
- removed C1, C2: 47uF/16V, Capacitor_SMD:C_1210_3225Metric, symbol pspice:C
- U1: value AD009-06H -> HB1531E; symbol ktRMT_Thumb:AD009-06H -> ktRMT_Thumb:HB1531E
Connections:
- net at SW1.1: now also U1.12 (PD2); no longer U1.6 (PA0)
- net at SW1.2: now also U1.11 (PD3); no longer U1.5 (PA1)
- net at U1.10 (PB0): now also SW2.1
- net at U1.3 (PA3/VPP): no longer SW2.2
- net at U1.4 (PA2): no longer SW2.1
- net at U1.9 (PB1): now also SW2.2
Changed lines of the file:
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@@
   (title_block
     (title "ktRMT_Thumb")
-    (date "2024-12-16")
-    (rev "0.1")
+    (date "2025-01-12")
+    (rev "0.2")
     (company "kt")
     (comment 1 "Infrared Learning Remote Controler")
-    (comment 2 "Use AD009-06H")
+    (comment 2 "Use HB1531")
     (comment 3 "Thumb type")
   )
-  (junction (at 157.48 104.14) (diameter 0) (color 0 0 0 0)
-  )
-  (junction (at 134.62 88.9) (diameter 0) (color 0 0 0 0)
-  )
-  (junction (at 157.48 67.31) (diameter 0) (color 0 0 0 0)
-  )
   (junction (at 205.74 83.82) (diameter 0) (color 0 0 0 0)
   )
   (junction (at 186.69 83.82) (diameter 0) (color 0 0 0 0)
   )
-  (wire (pts (xy 114.3 88.9) (xy 134.62 88.9))
-    (stroke (width 0) (type default) (color 0 0 0 0))
-  )
-  (wire (pts (xy 114.3 92.71) (xy 114.3 88.9))
+  (wire (pts (xy 208.28 114.3) (xy 208.28 144.78))
     (stroke (width 0) (type default) (color 0 0 0 0))
   )
@@
     (stroke (width 0) (type default) (color 0 0 0 0))
   )
-  (wire (pts (xy 157.48 62.23) (xy 157.48 67.31))
-    (stroke (width 0) (type default) (color 0 0 0 0))
-  )
-  (wire (pts (xy 161.29 116.84) (xy 43.18 116.84))
-    (stroke (width 0) (type default) (color 0 0 0 0))
-  )
-  (wire (pts (xy 134.62 104.14) (xy 157.48 104.14))
+  (wire (pts (xy 157.48 62.23) (xy 157.48 73.66))
+    (stroke (width 0) (type default) (color 0 0 0 0))
+  )
+  (wire (pts (xy 181.61 121.92) (xy 194.31 121.92))
     (stroke (width 0) (type default) (color 0 0 0 0))
   )
@@
     (stroke (width 0) (type default) (color 0 0 0 0))
   )
-  (wire (pts (xy 134.62 67.31) (xy 157.48 67.31))
-    (stroke (width 0) (type default) (color 0 0 0 0))
-  )
-  (wire (pts (xy 134.62 71.12) (xy 134.62 67.31))
+  (wire (pts (xy 138.43 134.62) (xy 138.43 109.22))
+    (stroke (width 0) (type default) (color 0 0 0 0))
+  )
+  (wire (pts (xy 181.61 116.84) (xy 205.74 116.84))
     (stroke (width 0) (type default) (color 0 0 0 0))
   )
@@
     (stroke (width 0) (type default) (color 0 0 0 0))
   )
-  (wire (pts (xy 91.44 109.22) (xy 161.29 109.22))
+  (wire (pts (xy 91.44 109.22) (xy 138.43 109.22))
+    (stroke (width 0) (type default) (color 0 0 0 0))
+  )
+  (wire (pts (xy 181.61 114.3) (xy 208.28 114.3))
     (stroke (width 0) (type default) (color 0 0 0 0))
   )
@@
     (stroke (width 0) (type default) (color 0 0 0 0))
   )
+  (wire (pts (xy 196.85 137.16) (xy 135.89 137.16))
+    (stroke (width 0) (type default) (color 0 0 0 0))
+  )
+  (wire (pts (xy 135.89 111.76) (xy 135.89 137.16))
+    (stroke (width 0) (type default) (color 0 0 0 0))
+  )
   (wire (pts (xy 186.69 83.82) (xy 186.69 104.14))
     (stroke (width 0) (type default) (color 0 0 0 0))
   )
-  (wire (pts (xy 134.62 83.82) (xy 134.62 88.9))
+  (wire (pts (xy 128.27 114.3) (xy 59.69 114.3))
     (stroke (width 0) (type default) (color 0 0 0 0))
   )
@@
     (stroke (width 0) (type default) (color 0 0 0 0))
   )
+  (wire (pts (xy 125.73 116.84) (xy 125.73 144.78))
+    (stroke (width 0) (type default) (color 0 0 0 0))
+  )
   (wire (pts (xy 72.39 109.22) (xy 81.28 109.22))
     (stroke (width 0) (type default) (color 0 0 0 0))
   )
-  (wire (pts (xy 157.48 67.31) (xy 157.48 73.66))
-    (stroke (width 0) (type default) (color 0 0 0 0))
-  )
-  (wire (pts (xy 161.29 114.3) (xy 59.69 114.3))
+  (wire (pts (xy 128.27 114.3) (xy 128.27 142.24))
+    (stroke (width 0) (type default) (color 0 0 0 0))
+  )
+  (wire (pts (xy 194.31 134.62) (xy 138.43 134.62))
+    (stroke (width 0) (type default) (color 0 0 0 0))
+  )
+  (wire (pts (xy 208.28 144.78) (xy 125.73 144.78))
     (stroke (width 0) (type default) (color 0 0 0 0))
   )
@@
     (stroke (width 0) (type default) (color 0 0 0 0))
   )
+  (wire (pts (xy 196.85 119.38) (xy 196.85 137.16))
+    (stroke (width 0) (type default) (color 0 0 0 0))
+  )
   (wire (pts (xy 186.69 62.23) (xy 186.69 83.82))
     (stroke (width 0) (type default) (color 0 0 0 0))
   )
+  (wire (pts (xy 181.61 119.38) (xy 196.85 119.38))
+    (stroke (width 0) (type default) (color 0 0 0 0))
+  )
   (wire (pts (xy 157.48 81.28) (xy 157.48 104.14))
     (stroke (width 0) (type default) (color 0 0 0 0))
   )
-  (wire (pts (xy 161.29 111.76) (xy 72.39 111.76))
-    (stroke (width 0) (type default) (color 0 0 0 0))
-  )
   (wire (pts (xy 43.18 116.84) (xy 43.18 114.3))
     (stroke (width 0) (type default) (color 0 0 0 0))
@@
     (stroke (width 0) (type default) (color 0 0 0 0))
   )
+  (wire (pts (xy 194.31 121.92) (xy 194.31 134.62))
+    (stroke (width 0) (type default) (color 0 0 0 0))
+  )
   (wire (pts (xy 43.18 114.3) (xy 49.53 114.3))
     (stroke (width 0) (type default) (color 0 0 0 0))
   )
-  (wire (pts (xy 161.29 106.68) (xy 114.3 106.68))
-    (stroke (width 0) (type default) (color 0 0 0 0))
-  )
   (wire (pts (xy 181.61 109.22) (xy 226.06 109.22))
     (stroke (width 0) (type default) (color 0 0 0 0))
@@
     (stroke (width 0) (type default) (color 0 0 0 0))
   )
-  (wire (pts (xy 114.3 106.68) (xy 114.3 105.41))
+  (wire (pts (xy 205.74 116.84) (xy 205.74 142.24))
+    (stroke (width 0) (type default) (color 0 0 0 0))
+  )
+  (wire (pts (xy 125.73 116.84) (xy 43.18 116.84))
     (stroke (width 0) (type default) (color 0 0 0 0))
   )
@@
     (stroke (width 0) (type default) (color 0 0 0 0))
   )
-  (wire (pts (xy 134.62 88.9) (xy 134.62 104.14))
+  (wire (pts (xy 128.27 142.24) (xy 205.74 142.24))
     (stroke (width 0) (type default) (color 0 0 0 0))
   )
   (wire (pts (xy 157.48 62.23) (xy 186.69 62.23))
+    (stroke (width 0) (type default) (color 0 0 0 0))
+  )
+  (wire (pts (xy 135.89 111.76) (xy 72.39 111.76))
     (stroke (width 0) (type default) (color 0 0 0 0))
   )
@@
     (pin "2")
   )
-  (symbol (lib_id "ktRMT_Thumb:AD009-06H") (at 171.45 111.76 0) (unit 1)
+  (symbol (lib_id "ktRMT_Thumb:HB1531E") (at 171.45 111.76 0) (unit 1)
     (in_bom yes) (on_board yes) (fields_autoplaced)
     (property "Reference" "U1" (id 0) (at 171.45 96.52 0))
-    (property "Value" "AD009-06H" (id 1) (at 171.45 99.06 0))
+    (property "Value" "HB1531E" (id 1) (at 171.45 99.06 0))
     (property "Footprint" "Package_SO:SOP-16_3.9x9.9mm_P1.27mm" (id 2) (at 171.45 111.76 0)
       (effects (font (size 1.27 1.27)) hide)
@@
     (pin "2")
   )
-  (symbol (lib_id "pspice:C") (at 114.3 99.06 0) (unit 1)
-    (in_bom yes) (on_board yes) (fields_autoplaced)
-    (property "Reference" "C2" (id 0) (at 119.38 97.7899 0)
-      (effects (font (size 1.27 1.27)) (justify left))
-    )
-    (property "Value" "47uF/16V" (id 1) (at 119.38 100.3299 0)
-      (effects (font (size 1.27 1.27)) (justify left))
-    )
-    (property "Footprint" "Capacitor_SMD:C_1210_3225Metric" (id 2) (at 114.3 99.06 0)
-      (effects (font (size 1.27 1.27)) hide)
-    )
-    (property "Datasheet" "~" (id 3) (at 114.3 99.06 0)
-      (effects (font (size 1.27 1.27)) hide)
-    )
-    (pin "1")
-    (pin "2")
-  )
-  (symbol (lib_id "pspice:C") (at 134.62 77.47 0) (unit 1)
-    (in_bom yes) (on_board yes) (fields_autoplaced)
-    (property "Reference" "C1" (id 0) (at 139.7 76.1999 0)
-      (effects (font (size 1.27 1.27)) (justify left))
-    )
-    (property "Value" "47uF/16V" (id 1) (at 139.7 78.7399 0)
-      (effects (font (size 1.27 1.27)) (justify left))
-    )
-    (property "Footprint" "Capacitor_SMD:C_1210_3225Metric" (id 2) (at 134.62 77.47 0)
-      (effects (font (size 1.27 1.27)) hide)
-    )
-    (property "Datasheet" "~" (id 3) (at 134.62 77.47 0)
-      (effects (font (size 1.27 1.27)) hide)
-    )
-    (pin "1")
-    (pin "2")
-  )
   (symbol (lib_id "Switch:SW_Push") (at 86.36 109.22 0) (unit 1)
     (in_bom yes) (on_board yes) (fields_autoplaced)
@@
       (reference "BT1") (unit 1) (value "3V") (footprint "ktRMT_Thumb:CR16xx_Holder")
     )
-    (path "/e4f45d12-446e-40d1-9f8b-94301740fd6b"
-      (reference "C1") (unit 1) (value "47uF/16V") (footprint "Capacitor_SMD:C_1210_3225Metric")
-    )
-    (path "/d8f8f7b8-0104-4ca4-9827-196e3d9bedab"
-      (reference "C2") (unit 1) (value "47uF/16V") (footprint "Capacitor_SMD:C_1210_3225Metric")
-    )
     (path "/8dad99e5-97f4-4b14-a20d-ada93c6437b0"
       (reference "D2") (unit 1) (value "LED") (footprint "LED_SMD:LED_1206_3216Metric")
@@
     )
     (path "/b009e36a-406e-48af-b8de-447612f15cf1"
-      (reference "U1") (unit 1) (value "AD009-06H") (footprint "Package_SO:SOP-16_3.9x9.9mm_P1.27mm")
-    )
-  )
+      (reference "U1") (unit 1) (value "HB1531E") (footprint "Package_SO:SOP-16_3.9x9.9mm_P1.27mm")
+    )
+  )
